File: Kicad - Copy/brewery 3dp motherboard/12V_Buck_Conv.kicad_sch (KiCad schematic)
At the start: 30 parts, among them U4 LM25145RGYR, U7 DOZ45N03T, U8 DOZ45N03T

Commit message: did stuff
Parts:
- added C24: 10uF, Capacitor_SMD:C_1210_3225Metric, symbol Device:C_Small
- C11: footprint Capacitor_SMD:C_0603_1608Metric -> Capacitor_SMD:C_1210_3225Metric
- C27: footprint Capacitor_SMD:C_0402_1005Metric -> Capacitor_SMD:C_0603_1608Metric
- R42: footprint Resistor_SMD:R_0402_1005Metric -> Resistor_SMD:R_0603_1608Metric
Connections:
- net GND: now also C24.2; no longer R5.2
- new net: C24.1, R5.2
Changed lines of the file:
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@@
 	)
 	(junction
-		(at 58.42 76.2)
+		(at 120.65 104.14)
 		(diameter 0)
 		(color 0 0 0 0)
 	)
 	(junction
-		(at 120.65 104.14)
+		(at 80.01 78.74)
 		(diameter 0)
 		(color 0 0 0 0)
 	)
 	(junction
-		(at 80.01 78.74)
+		(at 58.42 59.69)
 		(diameter 0)
 		(color 0 0 0 0)
 	)
 	(junction
-		(at 58.42 59.69)
+		(at 58.42 76.2)
 		(diameter 0)
 		(color 0 0 0 0)
@@
 	(wire
 		(pts
-			(xy 58.42 66.04) (xy 58.42 76.2)
+			(xy 185.42 93.98) (xy 214.63 93.98)
 		)
 		(stroke
@@
 	(wire
 		(pts
-			(xy 185.42 93.98) (xy 214.63 93.98)
+			(xy 195.58 119.38) (xy 195.58 88.9)
 		)
 		(stroke
@@
 	(wire
 		(pts
-			(xy 195.58 119.38) (xy 195.58 88.9)
+			(xy 31.75 76.2) (xy 35.56 76.2)
 		)
 		(stroke
@@
 	(wire
 		(pts
-			(xy 31.75 76.2) (xy 35.56 76.2)
+			(xy 195.58 130.81) (xy 222.25 130.81)
 		)
 		(stroke
@@
 	(wire
 		(pts
-			(xy 195.58 130.81) (xy 222.25 130.81)
+			(xy 58.42 73.66) (xy 58.42 76.2)
+		)
+		(stroke
+			(width 0)
+			(type default)
+		)
+	)
+	(wire
+		(pts
+			(xy 58.42 76.2) (xy 67.31 76.2)
 		)
 		(stroke
@@
 	(wire
 		(pts
-			(xy 44.45 59.69) (xy 35.56 59.69)
+			(xy 58.42 66.04) (xy 58.42 68.58)
 		)
 		(stroke
@@
 	(wire
 		(pts
-			(xy 198.12 60.96) (xy 208.28 60.96)
+			(xy 44.45 59.69) (xy 35.56 59.69)
 		)
 		(stroke
@@
 	(wire
 		(pts
-			(xy 110.49 114.3) (xy 110.49 88.9)
+			(xy 198.12 60.96) (xy 208.28 60.96)
 		)
 		(stroke
@@
 	(wire
 		(pts
-			(xy 185.42 78.74) (xy 189.23 78.74)
+			(xy 110.49 114.3) (xy 110.49 88.9)
 		)
 		(stroke
@@
 	(wire
 		(pts
-			(xy 260.35 58.42) (xy 260.35 60.96)
+			(xy 185.42 78.74) (xy 189.23 78.74)
 		)
 		(stroke
@@
 	(wire
 		(pts
-			(xy 134.62 104.14) (xy 139.7 104.14)
+			(xy 260.35 58.42) (xy 260.35 60.96)
 		)
 		(stroke
@@
 	(wire
 		(pts
-			(xy 91.44 73.66) (xy 139.7 73.66)
+			(xy 134.62 104.14) (xy 139.7 104.14)
 		)
 		(stroke
@@
 	(wire
 		(pts
-			(xy 58.42 76.2) (xy 67.31 76.2)
+			(xy 91.44 73.66) (xy 139.7 73.66)
 		)
 		(stroke
@@
 			)
 		)
-		(property "Footprint" "Capacitor_SMD:C_0402_1005Metric"
+		(property "Footprint" "Capacitor_SMD:C_0603_1608Metric"
 			(at 191.77 78.74 0)
 			(hide yes)
@@
 	)
 	(symbol
+		(lib_id "Device:C_Small")
+		(at 58.42 71.12 0)
+		(unit 1)
+		(body_style 1)
+		(exclude_from_sim no)
+		(in_bom yes)
+		(on_board yes)
+		(in_pos_files yes)
+		(dnp no)
+		(property "Reference" "C24"
+			(at 60.452 69.85 0)
+			(show_name no)
+			(do_not_autoplace no)
+			(effects
+				(font
+					(size 1.27 1.27)
+				)
+				(justify left)
+			)
+		)
+		(property "Value" "10uF"
+			(at 60.452 72.39 0)
+			(show_name no)
+			(do_not_autoplace no)
+			(effects
+				(font
+					(size 1.27 1.27)
+				)
+				(justify left)
+			)
+		)
+		(property "Footprint" "Capacitor_SMD:C_1210_3225Metric"
+			(at 58.42 71.12 0)
+			(hide yes)
+			(show_name no)
+			(do_not_autoplace no)
+			(effects
+				(font
+					(size 1.27 1.27)
+				)
+			)
+		)
+		(property "Datasheet" ""
+			(at 58.42 71.12 0)
+			(hide yes)
+			(show_name no)
+			(do_not_autoplace no)
+			(effects
+				(font
+					(size 1.27 1.27)
+				)
+			)
+		)
+		(property "Description" "Unpolarized capacitor, small symbol"
+			(at 58.42 71.12 0)
+			(hide yes)
+			(show_name no)
+			(do_not_autoplace no)
+			(effects
+				(font
+					(size 1.27 1.27)
+				)
+			)
+		)
+		(pin "1"
+		)
+		(pin "2"
+		)
+		(instances
+			(project "brewery 3dp motherboard"
+				(path "/63771b13-dd98-4833-96bf-ef6b5d3ded40/b04a4fac-8004-4ef1-b594-4ab3d5b5088e"
+					(reference "C24")
+					(unit 1)
+				)
+			)
+		)
+	)
+	(symbol
 		(lib_id "Device:R_Small")
 		(at 248.92 86.36 180)
@@
 			)
 		)
-		(property "Footprint" "Capacitor_SMD:C_0603_1608Metric"
+		(property "Footprint" "Capacitor_SMD:C_1210_3225Metric"
 			(at 67.31 69.85 0)
 			(hide yes)
@@
 			)
 		)
-		(property "Footprint" "Resistor_SMD:R_0402_1005Metric"
+		(property "Footprint" "Resistor_SMD:R_0603_1608Metric"
 			(at 201.93 88.9 0)
 			(hide yes)

Commit message: DID STUFF
Parts:
- C40: footprint Capacitor_SMD:C_0603_1608Metric -> Capacitor_SMD:C_0402_1005Metric
Changed lines of the file:
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@@
 			)
 		)
-		(property "Footprint" "Capacitor_SMD:C_0603_1608Metric"
+		(property "Footprint" "Capacitor_SMD:C_0402_1005Metric"
 			(at 248.92 93.98 0)
 			(hide yes)
