File: Kicad - Copy/brewery 3dp motherboard/Fan controller.kicad_sch (KiCad schematic)
At the start: 6 parts, among them J28 jumpers, J29 JST-XH, U18 DOZ45N03T

Commit message: did stuff (uploading kicad bits)
Parts:
- R98, R99: footprint Resistor_SMD:R_0402_1005Metric -> Resistor_SMD:R_0603_1608Metric
Changed lines of the file:
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@@
 			)
 		)
-		(property "Footprint" "Resistor_SMD:R_0402_1005Metric"
+		(property "Footprint" "Resistor_SMD:R_0603_1608Metric"
 			(at 100.33 71.12 0)
 			(hide yes)
@@
 			)
 		)
-		(property "Footprint" "Resistor_SMD:R_0402_1005Metric"
+		(property "Footprint" "Resistor_SMD:R_0603_1608Metric"
 			(at 104.14 77.47 0)
 			(hide yes)

Commit message: DID STUFF
Parts:
- R98: value 100 -> 2k
- R99: value 10k -> 20k
Changed lines of the file:
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@@
 			)
 		)
-		(property "Value" "100"
+		(property "Value" "2k"
 			(at 100.33 68.58 90)
 			(show_name no)
@@
 			)
 		)
-		(property "Value" "10k"
+		(property "Value" "20k"
 			(at 99.568 78.74 0)
 			(show_name no)
