File: Kicad - Copy/brewery 3dp motherboard/brewery 3dp motherboard.kicad_pcb (KiCad board)
At the start: 4 copper layers, 189.1 x 280.6 mm, 331 parts, among them J1 power in, J11 USB_C_Receptacle_USB2.0_14P, J16 heater in, J2 JST-XH, J26 Screw_Terminal_01x02, J27 Screw_Terminal_01x02, J28 jumpers, J29 JST-XH, J3 JST-XH, J30 jumpers, J31 JST-XH, J32 jumpers, J33 JST-XH, J34 jumpers, J35 JST-XH, J36 jumpers, J37 JST-XH, J38 jumpers, J39 JST-XH, J4 JST-XH, J40 jumpers, J41 JST-XH, J42 jumpers, J43 JST-XH, J44 jumpers, J45 JST-XH, J46 jumpers, J47 JST-XH, J48 jumpers, J49 JST-XH, J5 JST-XH, J50 jumpers, J51 JST-XH, J52 JST-XH, J53 JST-XH, J54 JST-XH, J55 JST-XH, J56 JST-XH, J57 JST-XH, J58 JST-XH, J59 JST-XH, J6 Conn_01x03_Pin, J60 JST-XH, J61 JST-XH, J62 JST-XH, J63 JST-XH, J64 JST-XH, J65 JST-XH, J66 JST-XH, J67 JST-XH, J68 Screw_Terminal_01x02, J69 Screw_Terminal_01x02, SW1 SW_Push, SW2 SW_Push, U1 MCP6004, U10 DOZ45N03T, U11 USBLC6-2SC6, U14 STM32F407Z_E-G_Tx, U16 DOZ45N03T, U17 DOZ45N03T, U18 DOZ45N03T, U19 DOZ45N03T, U2 LM61430AFSQRJRRQ1, U20 DOZ45N03T, U21 DOZ45N03T, U22 DOZ45N03T, U23 DOZ45N03T, U24 DOZ45N03T, U25 DOZ45N03T, U26 DOZ45N03T, U27 DOZ45N03T, U28 DOZ45N03T, U29 DOZ45N03T, U30 MCP6004, U31 MCP6004, U32 MCP6004, U33 MCP6004, U34 DOZ45N03T, U35 DOZ45N03T, U4 LM25145RGYR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

Commit message: did stuff
Parts:
- added C24: 10uF, Capacitor_SMD:C_1210_3225Metric, F.Cu at (204.1, 250.4)
- C11, C12: footprint Capacitor_SMD:C_0603_1608Metric -> Capacitor_SMD:C_1210_3225Metric
- C16, C19, C30, C32, C34, C41, R13, R14, R20, R23, R26, R27, R45, R47, R55, R61, U5: moved to B.Cu
- C27: footprint Capacitor_SMD:C_0402_1005Metric -> Capacitor_SMD:C_0603_1608Metric
- C28: footprint Capacitor_SMD:C_0402_1005Metric -> Capacitor_SMD:C_0603_1608Metric; moved to B.Cu
- R42, R5, R6: footprint Resistor_SMD:R_0402_1005Metric -> Resistor_SMD:R_0603_1608Metric
- R43: footprint Resistor_SMD:R_0402_1005Metric -> Resistor_SMD:R_0603_1608Metric; moved to B.Cu
- moved L1 231.9 mm to (186.2, 242.5), turned to 0 degrees
- moved C22 223.4 mm to (196.1, 247.9), turned to 0 degrees
- moved C23 221.2 mm to (196.1, 255.8), turned to 0 degrees
- moved R21 217.0 mm to (547.9, 127.3)
- moved C14 217.0 mm to (545.0, 129.2)
- moved C26 217.0 mm to (545.0, 133.2)
- moved C3 217.0 mm to (541.0, 128.2)
- moved J6 217.0 mm to (541.2, 119.6)
- moved U2 217.0 mm to (553.0, 129.0)
- moved C10 217.0 mm to (541.0, 130.7)
- moved C13 217.0 mm to (545.0, 127.3)
- moved C17 217.0 mm to (545.0, 131.2)
- moved L3 217.0 mm to (549.1, 121.8)
- moved R40 217.0 mm to (547.9, 129.3)
- moved R41 217.0 mm to (547.9, 131.2)
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Connections:
- R5 pad 1: GND -> Net-(U7-Drain)
- R5 pad 2: Net-(U7-Drain) -> Net-(C24-Pad1)
- U4 pad V: GND -> (no net)
Routing:
- net Net-(U9-Drain): track 0.00 -> 18.2 mm
- net Net-(U4-SW): track 15.1 -> 0.00 mm
- net Net-(U10-Drain): track 0.00 -> 13.8 mm
- net Net-(C42-Pad1): track 13.2 -> 0.00 mm
- net Net-(U7-Drain): track 11.8 -> 0.00 mm
- net Net-(C43-Pad1): track 0.00 -> 11.2 mm
- net Net-(U4-FB): track 9.82 -> 0.00 mm
- net Net-(U4-VCC): track 9.71 -> 0.00 mm, vias 2 -> 0
- net Net-(U4-LO): track 8.61 -> 0.00 mm, vias 2 -> 0
- net Net-(U4-HO): track 6.79 -> 0.00 mm, vias 2 -> 0
- net Net-(U4-COMP): track 6.16 -> 0.00 mm
- net GND: track 56.7 -> 62.6 mm, vias 11 -> 2
- net Net-(U5-FB): track 0.00 -> 5.37 mm
- net Net-(U5-ILIM): track 0.00 -> 5.31 mm
- net Net-(U4-BST): track 3.83 -> 0.00 mm, vias 2 -> 0
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
Commit message: did stuff (uploading kicad bits)
Parts:
- added 12V: TestPoint_Pad_D1.5mm, TestPoint:TestPoint_Pad_D1.5mm, F.Cu at (351.0, 152.8)
- added 5V: TestPoint_Pad_D1.5mm, TestPoint:TestPoint_Pad_D1.5mm, F.Cu at (345.6, 134.0)
- added VBUS: TestPoint_Pad_D1.5mm, TestPoint:TestPoint_Pad_D1.5mm, F.Cu at (355.7, 153.4)
- added VBUS: TestPoint_Pad_D1.5mm, TestPoint:TestPoint_Pad_D1.5mm, F.Cu at (354.3, 158.2)
- C16, C19, C28, C30, C32, C34, C41, R13, R14, R20, R23, R26, R27, R43, R45, R47, R55, R61, U5: moved to F.Cu
- R100, R101, R102, R103, R104, R105, R106, R107, R108, R109, R110, R111, R112, R113, R114, R115, R116, R117, R118, R119, R120, R121, R82, R83, R98, R99: footprint Resistor_SMD:R_0402_1005Metric -> Resistor_SMD:R_0603_1608Metric
- moved R121 642.0 mm to (333.3, 98.1), turned to 180 degrees
- moved R120 641.8 mm to (333.3, 96.6), turned to 180 degrees
- moved R112 639.4 mm to (365.4, 98.9), turned to -90 degrees
- moved R113 638.5 mm to (367.8, 98.1), turned to 180 degrees
- moved U29 637.1 mm to (332.6, 99.3)
- moved U25 633.7 mm to (367.2, 99.3)
- moved J51 631.9 mm to (334.4, 106.9), turned to 180 degrees
- moved D32 629.0 mm to (336.4, 101.2), turned to -90 degrees
- moved J43 628.7 mm to (369.0, 106.9), turned to 180 degrees
- moved D28 625.4 mm to (371.0, 101.1), turned to -90 degrees
- moved J50 624.1 mm to (330.5, 114.4), turned to 90 degrees
- moved J42 621.0 mm to (365.1, 114.4), turned to 90 degrees
- moved R104 605.2 mm to (374.2, 98.9), turned to -90 degrees
- moved R105 604.2 mm to (376.5, 98.2), turned to 180 degrees
- moved R114 600.4 mm to (356.8, 98.9), turned to -90 degrees
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Routing:
- net GND: track 62.6 -> 318.8 mm, vias 2 -> 71
- net +3.3V: track 0.00 -> 215.4 mm, vias 0 -> 26
- net VBUS: track 13.8 -> 132.8 mm
- net Net-(C42-Pad1): track 0.00 -> 42.0 mm, vias 0 -> 1
- net Net-(U7-Drain): track 0.00 -> 33.7 mm
- net Net-(U4-SW): track 0.00 -> 32.8 mm
- net Net-(D34-A2): track 0.00 -> 25.2 mm
- net Net-(D43-A2): track 0.00 -> 24.8 mm
- net Net-(D35-A2): track 0.00 -> 24.5 mm
- net Net-(D42-A2): track 0.00 -> 24.0 mm
- net Net-(D29-A2): track 0.00 -> 22.7 mm
- net Net-(D28-A2): track 0.00 -> 22.6 mm
- net Net-(D26-A2): track 0.00 -> 22.6 mm
- net Net-(D30-A2): track 0.00 -> 22.6 mm
- net Net-(D38-A2): track 0.00 -> 22.6 mm
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- added copper zone on In1.Cu, net GND
Other:
- board size 189.1 x 280.6 mm -> 469.1 x 275.2 mm
- board text removed: "Cheap JLC limmit"

Commit message: DID STUFF
Parts:
- removed 5V: TestPoint_Pad_D1.5mm, TestPoint:TestPoint_Pad_D1.5mm
- added C35: 47uF, Capacitor_SMD:C_0805_2012Metric, F.Cu at (643.4, -10.2)
- added R94: 0Ohm, footprints:Milliohm HoT-2-4.5-11-I, B.Cu at (571.9, -73.3)
- C13: footprint Capacitor_SMD:C_0402_1005Metric -> Capacitor_SMD:C_1206_3216Metric; moved to B.Cu
- C14: footprint Capacitor_SMD:C_0402_1005Metric -> Capacitor_SMD:C_1206_3216Metric
- C40: footprint Capacitor_SMD:C_0603_1608Metric -> Capacitor_SMD:C_0402_1005Metric
- C46, C47, C52: footprint Capacitor_SMD:C_0402_1005Metric -> Capacitor_SMD:C_0603_1608Metric
- R100, R102, R104, R106, R108, R110, R112, R114, R116, R118, R120, R98: value 100 -> 2k
- R101, R103, R105, R107, R109, R111, R113, R115, R117, R119, R121, R99: value 10k -> 20k
- moved F2 288.2 mm to (571.0, -15.8)
- moved C13 278.5 mm to (639.7, -5.70), turned to 90 degrees
- moved J11 277.6 mm to (644.7, 17.1)
- moved C29 277.5 mm to (565.5, -4.14)
- moved U5 277.5 mm to (596.2, -8.65)
- moved U4 277.5 mm to (567.2, -0.98)
- moved C15 277.5 mm to (565.3, 2.59)
- moved C18 277.5 mm to (570.7, 0.63)
- moved C20 277.5 mm to (560.3, -2.39)
- moved C23 277.5 mm to (566.1, 8.28)
- moved C26 277.5 mm to (645.7, -4.81)
- moved C30 277.5 mm to (594.5, -11.7)
- moved C32 277.5 mm to (601.5, -7.02)
- moved C4 277.5 mm to (616.3, 8.29)
- moved C43 277.5 mm to (604.7, -16.2)
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- renumbered VBUS to GND
Connections:
- U14 pad 127: unconnected-(U14-PG12-Pad127) -> Fan1
- U14 pad 128: unconnected-(U14-PG13-Pad128) -> Fan2
- U14 pad 129: unconnected-(U14-PG14-Pad129) -> Fan3
- U14 pad 13: Thermistor1 -> Thermistor13
- U14 pad 133: unconnected-(U14-PB3-Pad133) -> Fan4
- U14 pad 134: unconnected-(U14-PB4-Pad134) -> Fan5
- U14 pad 135: unconnected-(U14-PB5-Pad135) -> Fan6
- U14 pad 136: unconnected-(U14-PB6-Pad136) -> Fan7
- U14 pad 137: unconnected-(U14-PB7-Pad137) -> Fan8
- U14 pad 139: Fan3 -> Fan9
- U14 pad 14: Thermistor2 -> Thermistor15
- U14 pad 140: Fan4 -> Fan10
- U14 pad 15: Thermistor3 -> Thermistor16
- U14 pad 18: Thermistor4 -> Thermistor14
- U14 pad 19: Thermistor5 -> Thermistor18
- U14 pad 20: Thermistor6 -> Thermistor17
- U14 pad 21: Thermistor7 -> Thermistor20
- U14 pad 22: Thermistor8 -> Thermistor19
- U14 pad 35: Thermistor15 -> Heater4
- U14 pad 36: Thermistor16 -> Heater3
- U14 pad 37: Thermistor17 -> unconnected-(U14-PA3-Pad37)
- U14 pad 4: Fan5 -> Fan12
- U14 pad 40: Thermistor18 -> Thermistor1
- U14 pad 41: Thermistor19 -> Thermistor3
- U14 pad 42: Thermistor20 -> Thermistor8
- U14 pad 43: Fan11 -> Thermistor6
- U14 pad 44: Thermistor13 -> Thermistor7
- U14 pad 45: Thermistor14 -> Thermistor2
- U14 pad 46: Fan12 -> Thermistor4
- U14 pad 47: Heater1 -> Thermistor5
- U14 pad 5: Fan6 -> Fan11
- U14 pad 60: Fan7 -> unconnected-(U14-PE9-Pad60)
- U14 pad 64: Fan8 -> unconnected-(U14-PE11-Pad64)
- U14 pad 66: Fan9 -> unconnected-(U14-PE13-Pad66)
- U14 pad 67: Fan10 -> unconnected-(U14-PE14-Pad67)
- U14 pad 69: unconnected-(U14-PB10-Pad69) -> Heater2
- U14 pad 70: unconnected-(U14-PB11-Pad70) -> Heater1
- U14 pad 81: Heater2 -> unconnected-(U14-PD12-Pad81)
- U14 pad 82: Heater3 -> unconnected-(U14-PD13-Pad82)
- U14 pad 85: Fan1 -> unconnected-(U14-PD14-Pad85)
- U14 pad 86: Fan2 -> unconnected-(U14-PD15-Pad86)
Routing:
- net +3.3V: track 215.4 -> 540.9 mm, vias 26 -> 33
- net Heater1: track 0.00 -> 117.1 mm, vias 0 -> 2
- net Fan12: track 0.00 -> 115.2 mm, vias 0 -> 2
- net Fan11: track 0.00 -> 108.9 mm, vias 0 -> 2
- net Fan10: track 0.00 -> 105.5 mm, vias 0 -> 2
- net Fan9: track 0.00 -> 97.1 mm, vias 0 -> 2
- net Heater2: track 0.00 -> 95.7 mm, vias 0 -> 2
- net Fan8: track 0.00 -> 88.5 mm, vias 0 -> 2
- net Fan7: track 0.00 -> 80.0 mm, vias 0 -> 2
- net Fan6: track 0.00 -> 71.6 mm, vias 0 -> 2
- net Fan5: track 0.00 -> 63.5 mm, vias 0 -> 2
- net Thermistor14: track 0.00 -> 62.0 mm, vias 0 -> 2
- net Thermistor13: track 0.00 -> 61.9 mm
- net Thermistor6: track 0.00 -> 58.3 mm, vias 0 -> 2
- net Fan4: track 0.00 -> 54.9 mm, vias 0 -> 2
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- added copper zone on In1.Cu, net +12V
- added copper zone on In2.Cu, net +5V
- added copper zone on F.Cu, net Net-(U10-Drain)
- added copper zone on F.Cu, net Net-(U4-SW)
- added copper zone on B.Cu, net VBUS
- added copper zone on F.Cu, net VBUS
Other:
- board size 469.1 x 275.2 mm -> 234 x 100 mm
- board text removed: "Mellow D5"
