File: Kicad - Copy/brewery 3dp motherboard/brewery 3dp motherboard.kicad_sch (KiCad schematic)
At the start: 32 parts, among them J1 power in, J16 heater in, SW1 SW_Push, SW2 SW_Push, U14 STM32F407Z_E-G_Tx

Commit message: DID STUFF
Parts:
- added R94: 0Ohm, footprints:Milliohm HoT-2-4.5-11-I, symbol Device:R_Small
- C46, C47, C52: footprint Capacitor_SMD:C_0402_1005Metric -> Capacitor_SMD:C_0805_2012Metric
- R28, R30: value 100 -> 2k
- R29: value 4.7k -> 20k
- R82, R83: value 22 -> 43; footprint Resistor_SMD:R_0402_1005Metric -> Resistor_SMD:R_0603_1608Metric
Connections:
- net Fan1: now also U14.127 (PG12); no longer U14.85 (PD14)
- net Fan10: now also U14.140 (PB9); no longer U14.67 (PE14)
- net Fan11: now also U14.5 (PE6); no longer U14.43 (PA7)
- net Fan12: now also U14.4 (PE5); no longer U14.46 (PB0)
- net Fan2: now also U14.128 (PG13); no longer U14.86 (PD15)
- net Fan3: now also U14.129 (PG14); no longer U14.139 (PB8)
- net Fan4: now also U14.133 (PB3); no longer U14.140 (PB9)
- net Fan5: now also U14.134 (PB4); no longer U14.4 (PE5)
- net Fan6: now also U14.135 (PB5); no longer U14.5 (PE6)
- net Fan7: now also U14.136 (PB6); no longer U14.60 (PE9)
- net Fan8: now also U14.137 (PB7); no longer U14.64 (PE11)
- net Fan9: now also U14.139 (PB8); no longer U14.66 (PE13)
- net GND: now also R94.1, R94.2
- net Heater1: now also U14.70 (PB11); no longer U14.47 (PB1)
- net Heater2: now also U14.69 (PB10); no longer U14.81 (PD12)
- net Heater3: now also U14.36 (PA2); no longer U14.82 (PD13)
- net Heater4: now also U14.35 (PA1)
- net Thermistor1: now also U14.40 (PA4); no longer U14.13 (PF3)
- net Thermistor13: now also U14.13 (PF3); no longer U14.44 (PC4)
- net Thermistor14: now also U14.18 (PF6); no longer U14.45 (PC5)
- net Thermistor15: now also U14.14 (PF4); no longer U14.35 (PA1)
- net Thermistor16: now also U14.15 (PF5); no longer U14.36 (PA2)
- net Thermistor17: now also U14.20 (PF8); no longer U14.37 (PA3)
- net Thermistor18: now also U14.19 (PF7); no longer U14.40 (PA4)
- net Thermistor19: now also U14.22 (PF10); no longer U14.41 (PA5)
- net Thermistor2: now also U14.45 (PC5); no longer U14.14 (PF4)
- net Thermistor20: now also U14.21 (PF9); no longer U14.42 (PA6)
- net Thermistor3: now also U14.41 (PA5); no longer U14.15 (PF5)
- net Thermistor4: now also U14.46 (PB0); no longer U14.18 (PF6)
- net Thermistor5: now also U14.47 (PB1); no longer U14.19 (PF7)
- net Thermistor6: now also U14.43 (PA7); no longer U14.20 (PF8)
- net Thermistor7: now also U14.44 (PC4); no longer U14.21 (PF9)
- net Thermistor8: now also U14.42 (PA6); no longer U14.22 (PF10)
