File: Kicad/brewery 3dp motherboard/brewery 3dp motherboard.kicad_pcb (KiCad board)
At the start: 4 copper layers, 189.1 x 280.6 mm, 331 parts, among them J1 power in, J11 USB_C_Receptacle_USB2.0_14P, J16 heater in, J2 JST-XH, J26 Screw_Terminal_01x02, J27 Screw_Terminal_01x02, J28 jumpers, J29 JST-XH, J3 JST-XH, J30 jumpers, J31 JST-XH, J32 jumpers, J33 JST-XH, J34 jumpers, J35 JST-XH, J36 jumpers, J37 JST-XH, J38 jumpers, J39 JST-XH, J4 JST-XH, J40 jumpers, J41 JST-XH, J42 jumpers, J43 JST-XH, J44 jumpers, J45 JST-XH, J46 jumpers, J47 JST-XH, J48 jumpers, J49 JST-XH, J5 JST-XH, J50 jumpers, J51 JST-XH, J52 JST-XH, J53 JST-XH, J54 JST-XH, J55 JST-XH, J56 JST-XH, J57 JST-XH, J58 JST-XH, J59 JST-XH, J6 Conn_01x03_Pin, J60 JST-XH, J61 JST-XH, J62 JST-XH, J63 JST-XH, J64 JST-XH, J65 JST-XH, J66 JST-XH, J67 JST-XH, J68 Screw_Terminal_01x02, J69 Screw_Terminal_01x02, SW1 SW_Push, SW2 SW_Push, U1 MCP6004, U10 DOZ45N03T, U11 USBLC6-2SC6, U14 STM32F407Z_E-G_Tx, U16 DOZ45N03T, U17 DOZ45N03T, U18 DOZ45N03T, U19 DOZ45N03T, U2 LM61430AFSQRJRRQ1, U20 DOZ45N03T, U21 DOZ45N03T, U22 DOZ45N03T, U23 DOZ45N03T, U24 DOZ45N03T, U25 DOZ45N03T, U26 DOZ45N03T, U27 DOZ45N03T, U28 DOZ45N03T, U29 DOZ45N03T, U30 MCP6004, U31 MCP6004, U32 MCP6004, U33 MCP6004, U34 DOZ45N03T, U35 DOZ45N03T, U4 LM25145RGYR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

Commit message: cleaned up structure a bit
Parts:
- added 12V: TestPoint_Pad_D1.5mm, TestPoint:TestPoint_Pad_D1.5mm, F.Cu at (584.8, 3.51)
- added C24: 10uF, Capacitor_SMD:C_1210_3225Metric, F.Cu at (583.1, 10.1)
- added C35: 47uF, Capacitor_SMD:C_0805_2012Metric, F.Cu at (643.4, -10.2)
- added GND: TestPoint_Pad_D1.5mm, TestPoint:TestPoint_Pad_D1.5mm, F.Cu at (588.2, 8.86)
- added R94: 0Ohm, footprints:Milliohm HoT-2-4.5-11-I, B.Cu at (571.9, -73.3)
- added VBUS: TestPoint_Pad_D1.5mm, TestPoint:TestPoint_Pad_D1.5mm, F.Cu at (589.6, 4.09)
- C11, C12: footprint Capacitor_SMD:C_0603_1608Metric -> Capacitor_SMD:C_1210_3225Metric
- C13: footprint Capacitor_SMD:C_0402_1005Metric -> Capacitor_SMD:C_1206_3216Metric; moved to B.Cu
- C14: footprint Capacitor_SMD:C_0402_1005Metric -> Capacitor_SMD:C_1206_3216Metric
- C27, C28, C46, C47, C52: footprint Capacitor_SMD:C_0402_1005Metric -> Capacitor_SMD:C_0603_1608Metric
- C40: footprint Capacitor_SMD:C_0603_1608Metric -> Capacitor_SMD:C_0402_1005Metric
- R100, R102, R104, R106, R108, R110, R112, R114, R116, R118, R120, R98: value 100 -> 2k; footprint Resistor_SMD:R_0402_1005Metric -> Resistor_SMD:R_0603_1608Metric
- R101, R103, R105, R107, R109, R111, R113, R115, R117, R119, R121, R99: value 10k -> 20k; footprint Resistor_SMD:R_0402_1005Metric -> Resistor_SMD:R_0603_1608Metric
- R42, R43, R5, R6, R82, R83: footprint Resistor_SMD:R_0402_1005Metric -> Resistor_SMD:R_0603_1608Metric
- moved R121 421.8 mm to (567.1, -51.2), turned to 180 degrees
- moved R120 421.4 mm to (567.1, -52.8), turned to 180 degrees
- moved U29 417.1 mm to (566.5, -50.0)
- moved D32 413.5 mm to (570.2, -48.2), turned to -90 degrees
- moved R113 411.3 mm to (601.7, -51.2), turned to 180 degrees
- moved R112 410.0 mm to (599.3, -50.4), turned to -90 degrees
- moved U25 406.6 mm to (601.0, -50.0)
- moved J51 406.0 mm to (568.3, -42.4), turned to 180 degrees
- moved D28 402.8 mm to (604.9, -48.2), turned to -90 degrees
- moved J50 396.4 mm to (564.4, -34.9), turned to 90 degrees
- moved J43 395.7 mm to (602.8, -42.4), turned to 180 degrees
- moved R109 391.1 mm to (636.2, -51.2), turned to 180 degrees
- moved R108 388.5 mm to (633.9, -50.4), turned to -90 degrees
- moved D26 387.8 mm to (639.4, -48.2), turned to -90 degrees
- moved U23 387.5 mm to (635.6, -50.0)
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Connections:
- R5 pad 1: GND -> Net-(U7-Drain)
- R5 pad 2: Net-(U7-Drain) -> Net-(C24-Pad1)
- U14 pad 127: unconnected-(U14-PG12-Pad127) -> Fan1
- U14 pad 128: unconnected-(U14-PG13-Pad128) -> Fan2
- U14 pad 129: unconnected-(U14-PG14-Pad129) -> Fan3
- U14 pad 13: Thermistor1 -> Thermistor13
- U14 pad 133: unconnected-(U14-PB3-Pad133) -> Fan4
- U14 pad 134: unconnected-(U14-PB4-Pad134) -> Fan5
- U14 pad 135: unconnected-(U14-PB5-Pad135) -> Fan6
- U14 pad 136: unconnected-(U14-PB6-Pad136) -> Fan7
- U14 pad 137: unconnected-(U14-PB7-Pad137) -> Fan8
- U14 pad 139: Fan3 -> Fan9
- U14 pad 14: Thermistor2 -> Thermistor15
- U14 pad 140: Fan4 -> Fan10
- U14 pad 15: Thermistor3 -> Thermistor16
- U14 pad 18: Thermistor4 -> Thermistor14
- U14 pad 19: Thermistor5 -> Thermistor18
- U14 pad 20: Thermistor6 -> Thermistor17
- U14 pad 21: Thermistor7 -> Thermistor20
- U14 pad 22: Thermistor8 -> Thermistor19
- U14 pad 35: Thermistor15 -> Heater4
- U14 pad 36: Thermistor16 -> Heater3
- U14 pad 37: Thermistor17 -> unconnected-(U14-PA3-Pad37)
- U14 pad 4: Fan5 -> Fan12
- U14 pad 40: Thermistor18 -> Thermistor1
- U14 pad 41: Thermistor19 -> Thermistor3
- U14 pad 42: Thermistor20 -> Thermistor8
- U14 pad 43: Fan11 -> Thermistor6
- U14 pad 44: Thermistor13 -> Thermistor7
- U14 pad 45: Thermistor14 -> Thermistor2
- U14 pad 46: Fan12 -> Thermistor4
- U14 pad 47: Heater1 -> Thermistor5
- U14 pad 5: Fan6 -> Fan11
- U14 pad 60: Fan7 -> unconnected-(U14-PE9-Pad60)
- U14 pad 64: Fan8 -> unconnected-(U14-PE11-Pad64)
- U14 pad 66: Fan9 -> unconnected-(U14-PE13-Pad66)
- U14 pad 67: Fan10 -> unconnected-(U14-PE14-Pad67)
- U14 pad 69: unconnected-(U14-PB10-Pad69) -> Heater2
- U14 pad 70: unconnected-(U14-PB11-Pad70) -> Heater1
- U14 pad 81: Heater2 -> unconnected-(U14-PD12-Pad81)
- U14 pad 82: Heater3 -> unconnected-(U14-PD13-Pad82)
- U14 pad 85: Fan1 -> unconnected-(U14-PD14-Pad85)
- U14 pad 86: Fan2 -> unconnected-(U14-PD15-Pad86)
Routing:
- net +3.3V: track 0.00 -> 540.9 mm, vias 0 -> 33
- net GND: track 56.7 -> 290.8 mm, vias 11 -> 207
- net Heater1: track 0.00 -> 117.1 mm, vias 0 -> 2
- net Fan12: track 0.00 -> 115.2 mm, vias 0 -> 2
- net Fan11: track 0.00 -> 108.9 mm, vias 0 -> 2
- net Fan10: track 0.00 -> 105.5 mm, vias 0 -> 2
- net Fan9: track 0.00 -> 97.1 mm, vias 0 -> 2
- net VBUS: track 17.3 -> 113.1 mm, vias 0 -> 25
- net Heater2: track 0.00 -> 95.7 mm, vias 0 -> 2
- net Fan8: track 0.00 -> 88.5 mm, vias 0 -> 2
- net Fan7: track 0.00 -> 80.0 mm, vias 0 -> 2
- net Fan6: track 0.00 -> 71.6 mm, vias 0 -> 2
- net Fan5: track 0.00 -> 63.5 mm, vias 0 -> 2
- net Thermistor14: track 0.00 -> 62.0 mm, vias 0 -> 2
- net Thermistor13: track 0.00 -> 61.9 mm
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- added copper zone on In1.Cu, net +12V
- added copper zone on In2.Cu, net +5V
- added copper zone on In1.Cu, net GND
- added copper zone on F.Cu, net Net-(U10-Drain)
- added copper zone on F.Cu, net Net-(U4-SW)
- added copper zone on B.Cu, net VBUS
- added copper zone on F.Cu, net VBUS
Other:
- board size 189.1 x 280.6 mm -> 234 x 100 mm
- board text removed: "Cheap JLC limmit"
- board text removed: "Mellow D5"
