File: Kicad/brewery 3dp motherboard/brewery 3dp motherboard.kicad_pcb (KiCad board)
At the start: 4 copper layers, 234 x 100 mm, 337 parts, among them J1 power in, J11 USB_C_Receptacle_USB2.0_14P, J16 heater in, J2 JST-XH, J26 Screw_Terminal_01x02, J27 Screw_Terminal_01x02, J28 jumpers, J29 JST-XH, J3 JST-XH, J30 jumpers, J31 JST-XH, J32 jumpers, J33 JST-XH, J34 jumpers, J35 JST-XH, J36 jumpers, J37 JST-XH, J38 jumpers, J39 JST-XH, J4 JST-XH, J40 jumpers, J41 JST-XH, J42 jumpers, J43 JST-XH, J44 jumpers, J45 JST-XH, J46 jumpers, J47 JST-XH, J48 jumpers, J49 JST-XH, J5 JST-XH, J50 jumpers, J51 JST-XH, J52 JST-XH, J53 JST-XH, J54 JST-XH, J55 JST-XH, J56 JST-XH, J57 JST-XH, J58 JST-XH, J59 JST-XH, J6 Conn_01x03_Pin, J60 JST-XH, J61 JST-XH, J62 JST-XH, J63 JST-XH, J64 JST-XH, J65 JST-XH, J66 JST-XH, J67 JST-XH, J68 Screw_Terminal_01x02, J69 Screw_Terminal_01x02, SW1 SW_Push, SW2 SW_Push, U1 MCP6004, U10 DOZ45N03T, U11 USBLC6-2SC6, U14 STM32F407Z_E-G_Tx, U16 DOZ45N03T, U17 DOZ45N03T, U18 DOZ45N03T, U19 DOZ45N03T, U2 LM61430AFSQRJRRQ1, U20 DOZ45N03T, U21 DOZ45N03T, U22 DOZ45N03T, U23 DOZ45N03T, U24 DOZ45N03T, U25 DOZ45N03T, U26 DOZ45N03T, U27 DOZ45N03T, U28 DOZ45N03T, U29 DOZ45N03T, U30 MCP6004, U31 MCP6004, U32 MCP6004, U33 MCP6004, U34 DOZ45N03T, U35 DOZ45N03T, U4 LM25145RGYR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

Commit message: stufffff
Parts:
- added G***: LOGO, LOGO, B.Cu at (65.2, 119.3)
- added G***: LOGO, LOGO, B.Cu at (81.1, 94.8)
- added G***: LOGO, LOGO, B.Cu at (146.6, 71.1)
- added G***: LOGO, LOGO, B.Cu at (83.0, 71.8)
- added G***: LOGO, LOGO, B.Cu at (154.8, 106.7)
- C46, C47, C52: footprint Capacitor_SMD:C_0603_1608Metric -> Capacitor_SMD:C_0805_2012Metric
- moved C67 522.5 mm to (165.1, 94.6)
- moved C46 521.9 mm to (138.6, 105.3)
- moved C15 521.1 mm to (58.3, 122.8)
- moved C20 521.1 mm to (53.3, 117.8)
- moved C23 521.1 mm to (59.1, 128.5)
- moved C30 521.1 mm to (87.5, 108.5)
- moved C31 521.1 mm to (65.5, 120.9)
- moved C32 521.1 mm to (94.5, 113.2)
- moved C54 521.1 mm to (165.5, 98.6)
- moved C55 521.1 mm to (140.0, 100.2)
- moved C56 521.1 mm to (155.1, 109.2)
- moved C59 521.1 mm to (140.0, 95.2)
- moved C75 521.1 mm to (169.6, 123.1)
- moved C77 521.1 mm to (172.3, 89.9)
- moved C9 521.1 mm to (161.0, 127.0)
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Connections:
- U4 pad GND: (no net) -> GND
- U5 pad GND: (no net) -> GND
Routing:
- net Net-(U14-VCAP_1): track 2.25 -> 2.94 mm
- net GND: track 290.8 -> 290.9 mm, vias 207 -> 209
Other:
- board size 234 x 100 mm -> 140 x 100 mm
- board text added: "Brewery V1.0 @WilliamPrime"
- board text added: "Flux goes here"
- board text added: "Hey this text is hot!"
- board text added: "Meow"
- board text added: "So, i know we put one cap here could you please try not to knock it off?"
- board text added: "dont knock me off"
- board text added: "now you've really broke it"
- board text removed: "Kai MX4"
