File: OLD/Kicad/brewery 3dp motherboard/heater.kicad_sch (KiCad schematic)
At the start: 6 parts, among them J26 Screw_Terminal_01x02, U16 DOZ45N03T

Commit message: cleaned up structure a bit
Parts:
- R80: value 2k -> 100
- R81: value 20k -> 10k
Other:
- moved on the sheet: R90
Changed lines of the file:
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@@
 	(paper "A4")
-	(junction
-		(at 77.47 27.94)
-		(diameter 0)
-		(color 0 0 0 0)
-	)
 	(junction
 		(at 80.01 62.23)
@@
 	(wire
 		(pts
+			(xy 77.47 36.83) (xy 77.47 40.64)
+		)
+		(stroke
+			(width 0)
+			(type default)
+		)
+	)
+	(wire
+		(pts
 			(xy 80.01 62.23) (xy 80.01 59.69)
 		)
@@
 	(wire
 		(pts
-			(xy 77.47 36.83) (xy 74.93 36.83)
-		)
-		(stroke
-			(width 0)
-			(type default)
-		)
-	)
-	(wire
-		(pts
-			(xy 77.47 27.94) (xy 77.47 36.83)
-		)
-		(stroke
-			(width 0)
-			(type default)
-		)
-	)
-	(wire
-		(pts
 			(xy 90.17 54.61) (xy 90.17 62.23)
 		)
@@
 	(wire
 		(pts
+			(xy 77.47 40.64) (xy 80.01 40.64)
+		)
+		(stroke
+			(width 0)
+			(type default)
+		)
+	)
+	(wire
+		(pts
 			(xy 64.77 50.8) (xy 66.04 50.8)
 		)
@@
 	(wire
 		(pts
-			(xy 74.93 27.94) (xy 77.47 27.94)
+			(xy 77.47 27.94) (xy 80.01 27.94)
 		)
 		(stroke
@@
 	(wire
 		(pts
-			(xy 77.47 27.94) (xy 80.01 27.94)
-		)
-		(stroke
-			(width 0)
-			(type default)
-		)
-	)
-	(wire
-		(pts
-			(xy 74.93 31.75) (xy 74.93 27.94)
+			(xy 77.47 31.75) (xy 77.47 27.94)
 		)
 		(stroke
@@
 			)
 		)
-		(property "Value" "20k"
+		(property "Value" "10k"
 			(at 61.468 58.42 0)
 			(show_name no)
@@
 			)
 		)
-		(property "Value" "2k"
+		(property "Value" "100"
 			(at 62.23 48.26 90)
 			(show_name no)
@@
 	(symbol
 		(lib_id "Device:R_Small")
-		(at 74.93 34.29 0)
+		(at 77.47 34.29 0)
 		(unit 1)
 		(body_style 1)
@@
 		(dnp no)
 		(property "Reference" "R90"
-			(at 68.58 32.512 0)
+			(at 71.12 32.512 0)
 			(show_name no)
 			(do_not_autoplace no)
@@
 		)
 		(property "Value" "0Ohm"
-			(at 73.66 34.798 0)
-			(show_name no)
-			(do_not_autoplace no)
-			(effects
-				(font
-					(size 1.27 1.27)
-				)
-				(justify right)
+			(at 71.12 35.052 0)
+			(show_name no)
+			(do_not_autoplace no)
+			(effects
+				(font
+					(size 1.27 1.27)
+				)
+				(justify left)
 			)
 		)
 		(property "Footprint" "footprints:Milliohm HoT-2-4.5-11-I"
-			(at 74.93 34.29 0)
+			(at 77.47 34.29 0)
 			(hide yes)
 			(show_name no)
@@
 		)
 		(property "Datasheet" ""
-			(at 74.93 34.29 0)
+			(at 77.47 34.29 0)
 			(hide yes)
 			(show_name no)
@@
 		)
 		(property "Description" "Resistor, small symbol"
-			(at 74.93 34.29 0)
-			(hide yes)
-			(show_name no)
+			(at 77.47 34.29 0)
+			(hide yes)
+			(show_name no)
